Commit message: Develop gazebo launch file, add inertias to urdf

File: routewise_ws/src/rw_description/rw_description/urdf/routewise_core.xacro (robot description, xacro)
@@ -7,4 +7,21 @@
     <xacro:property name="wheel_radius" value="0.075"/>
     <xacro:property name="wheel_width" value="0.05"/>
+    <!-- Inertial Macros -->
+    <xacro:macro name="inertial_box" params="mass x y z">
+        <inertial>
+            <mass value="${mass}"/>
+            <inertia ixx="${mass/12.0*(y*y + z*z)}" ixy="0.0" ixz="0.0"
+                     iyy="${mass/12.0*(x*x + z*z)}" iyz="0.0"
+                     izz="${mass/12.0*(x*x + y*y)}"/>
+        </inertial>
+    </xacro:macro>
+    <xacro:macro name="inertial_cylinder" params="mass r h">
+        <inertial>
+            <mass value="${mass}"/>
+            <inertia ixx="${(1/4.0)*mass*r*r + (1/12.0)*mass*h*h}" ixy="0.0" ixz="0.0"
+                     iyy="${(1/4.0)*mass*r*r + (1/12.0)*mass*h*h}" iyz="0.0"
+                     izz="${(1/2.0)*mass*r*r}"/>
+        </inertial>
+    </xacro:macro>
     <!-- Base Link -->
     <link name="base_link">
@@ -20,4 +37,5 @@
             </geometry>
         </collision>
+        <xacro:inertial_box mass="10.0" x="${base_length}" y="${base_width}" z="${base_height}"/>
     </link>
     <!-- Wheel Link Macro -->
@@ -35,4 +53,5 @@
                 </geometry>
             </collision>
+            <xacro:inertial_cylinder mass="2.0" r="${wheel_radius}" h="${wheel_width}"/>
         </link>
     </xacro:macro>
@@ -42,5 +61,5 @@
             <parent link="${parent}"/>
             <child link="${child}"/>
-            <origin xyz="${xyz}" rpy="0 0 0"/>
+            <origin xyz="${xyz}" rpy="0 1.57 0"/>
             <axis xyz="0 0 1"/>
         </joint>

Commit message: Develop mecanum_wheel.xacro with all links and joints

File: routewise_ws/src/rw_description/rw_description/urdf/routewise_core.xacro (robot description, xacro)
@@ -61,5 +61,5 @@
             <parent link="${parent}"/>
             <child link="${child}"/>
-            <origin xyz="${xyz}" rpy="0 1.57 0"/>
+            <origin xyz="${xyz}" rpy="0 0 0"/>
             <axis xyz="0 0 1"/>
         </joint>
