Commit message: Reorient rollers on wheels, integrate mecanum wheels to robot

File: routewise_ws/src/rw_description/rw_description/urdf/mecanum_wheel.xacro (robot description, xacro)
@@ -1,12 +1,19 @@
 <?xml version="1.0"?>
 <robot xmlns:xacro="http://ros.org/wiki/xacro">
+  <!-- Properties -->
+  <xacro:property name="wheel_mass" value="2.0"/> <!-- Assume a mass for the wheel -->
+  <xacro:property name="roller_mass" value="0.1"/> <!-- Assume a mass for the rollers -->
+  <xacro:property name="wheel_radius" value="0.1"/>
+  <xacro:property name="wheel_width" value="0.05"/>
+  <xacro:property name="roller_radius" value="0.02"/>
+  <xacro:property name="roller_length" value="0.05"/>
+  <xacro:property name="roller_angle" value="0.785398"/> <!-- 45 degrees in radians -->
   <!-- Mecanum Wheel Macro -->
   <xacro:macro name="mecanum_wheel" params="name">
-    <!-- Properties -->
-    <xacro:property name="wheel_radius" value="0.1"/>
-    <xacro:property name="wheel_width" value="0.05"/>
-    <xacro:property name="roller_radius" value="0.02"/>
-    <xacro:property name="roller_length" value="0.05"/>
-    <xacro:property name="roller_angle" value="0.785398"/> <!-- 45 degrees in radians -->
+    <!-- Derived Properties -->
+    <xacro:property name="I_wheel_xx_yy" value="0.0250833333333333"/>
+    <xacro:property name="I_wheel_zz" value="0.0100000000000000"/>
+    <xacro:property name="I_roller_xx_yy" value="0.0008750000000000"/>
+    <xacro:property name="I_roller_zz" value="0.0002000000000000"/>
     <!-- Main Wheel Body -->
     <link name="${name}">
@@ -21,33 +28,47 @@
         </geometry>
       </collision>
+      <inertial>
+        <mass value="${wheel_mass}"/>
+        <inertia ixx="${I_wheel_xx_yy}" ixy="0" ixz="0" iyy="${I_wheel_xx_yy}" iyz="0" izz="${I_wheel_zz}"/>
+      </inertial>
     </link>
-    <!-- Roller Macro -->
-    <xacro:macro name="roller" params="name angle">
-      <link name="${name}">
-        <visual>
-          <geometry>
-            <cylinder radius="${roller_radius}" length="${roller_length}"/>
-          </geometry>
-        </visual>
-        <collision>
-          <geometry>
-            <cylinder radius="${roller_radius}" length="${roller_length}"/>
-          </geometry>
-        </collision>
-      </link>
-      <joint name="${name}_joint" type="continuous">
-        <parent link="${name}"/>
-        <child link="${name}"/>
-        <origin rpy="0 0 ${angle}" xyz="0 0 0"/>
-        <axis xyz="0 0 1"/>
-      </joint>
-    </xacro:macro>
+  <!-- Roller Macro -->
+  <xacro:macro name="roller" params="name parent angle">
+    <link name="${name}">
+      <visual>
+        <geometry>
+          <cylinder radius="${roller_radius}" length="${roller_length}"/>
+        </geometry>
+      </visual>
+      <collision>
+        <geometry>
+          <cylinder radius="${roller_radius}" length="${roller_length}"/>
+        </geometry>
+      </collision>
+      <inertial>
+        <mass value="${roller_mass}"/>
+        <inertia ixx="${I_roller_xx_yy}" ixy="0" ixz="0" iyy="${I_roller_xx_yy}" iyz="0" izz="${I_roller_zz}"/>
+      </inertial>
+    </link>
+    <joint name="${name}_joint" type="continuous">
+      <parent link="${parent}"/>
+      <child link="${name}"/>
+      <origin
+          xyz="${wheel_radius*cos(angle)} ${wheel_radius*sin(angle)} 0"
+          rpy="${roller_angle} 0 ${angle}"/>
+      <axis xyz="0 0 1"/>
+   </joint>
+  </xacro:macro>
     <!-- Rollers -->
-    <xacro:roller name="${name}_roller_1" angle="0"/>
-    <xacro:roller name="${name}_roller_2" angle="${2*pi/3}"/>
-    <xacro:roller name="${name}_roller_3" angle="${4*pi/3}"/>
-    <xacro:roller name="${name}_roller_4" angle="${pi/6}"/>
-    <xacro:roller name="${name}_roller_5" angle="${pi/2 + pi/6}"/>
-    <xacro:roller name="${name}_roller_6" angle="${pi + pi/6}"/>
+    <xacro:roller name="${name}_roller_1" parent="${name}" angle="0"/>
+    <xacro:roller name="${name}_roller_2" parent="${name}" angle="${1*2*pi/10}"/>
+    <xacro:roller name="${name}_roller_3" parent="${name}" angle="${2*2*pi/10}"/>
+    <xacro:roller name="${name}_roller_4" parent="${name}" angle="${3*2*pi/10}"/>
+    <xacro:roller name="${name}_roller_5" parent="${name}" angle="${4*2*pi/10}"/>
+    <xacro:roller name="${name}_roller_6" parent="${name}" angle="${5*2*pi/10}"/>
+    <xacro:roller name="${name}_roller_7" parent="${name}" angle="${6*2*pi/10}"/>
+    <xacro:roller name="${name}_roller_8" parent="${name}" angle="${7*2*pi/10}"/>
+    <xacro:roller name="${name}_roller_9" parent="${name}" angle="${8*2*pi/10}"/>
+    <xacro:roller name="${name}_roller_10" parent="${name}" angle="${9*2*pi/10}"/>
   </xacro:macro>
 </robot>

File: routewise_ws/src/rw_description/rw_description/urdf/routewise.urdf.xacro (robot description, xacro)
@@ -2,4 +2,5 @@
 <robot xmlns:xacro="http://ros.org/wiki/xacro" name="routewise">
     <!-- Include Material and Core Files -->
+    <xacro:include filename="$(find rw_description)/urdf/mecanum_wheel.xacro"/>
     <xacro:include filename="$(find rw_description)/urdf/routewise_material.xacro"/>
     <xacro:include filename="$(find rw_description)/urdf/routewise_core.xacro"/>

File: routewise_ws/src/rw_description/rw_description/urdf/routewise_core.xacro (robot description, xacro)
@@ -5,6 +5,4 @@
     <xacro:property name="base_width" value="0.5"/>
     <xacro:property name="base_height" value="0.1"/>
-    <xacro:property name="wheel_radius" value="0.075"/>
-    <xacro:property name="wheel_width" value="0.05"/>
     <!-- Inertial Macros -->
     <xacro:macro name="inertial_box" params="mass x y z">
@@ -39,21 +37,4 @@
         <xacro:inertial_box mass="10.0" x="${base_length}" y="${base_width}" z="${base_height}"/>
     </link>
-    <!-- Wheel Link Macro -->
-    <xacro:macro name="wheel_link" params="name">
-        <link name="${name}">
-            <visual>
-                <geometry>
-                    <cylinder radius="${wheel_radius}" length="${wheel_width}"/>
-                </geometry>
-                <material name="grey"/>
-            </visual>
-            <collision>
-                <geometry>
-                    <cylinder radius="${wheel_radius}" length="${wheel_width}"/>
-                </geometry>
-            </collision>
-            <xacro:inertial_cylinder mass="2.0" r="${wheel_radius}" h="${wheel_width}"/>
-        </link>
-    </xacro:macro>
     <!-- Wheel Joint Macro -->
     <xacro:macro name="wheel_joint" params="name parent child xyz">
@@ -61,13 +42,13 @@
             <parent link="${parent}"/>
             <child link="${child}"/>
-            <origin xyz="${xyz}" rpy="0 0 0"/>
+            <origin xyz="${xyz}" rpy="${pi/2} 0 0"/>
             <axis xyz="0 0 1"/>
         </joint>
     </xacro:macro>
     <!-- Wheel Links and Joints -->
-    <xacro:wheel_link name="front_left_wheel"/>
-    <xacro:wheel_link name="front_right_wheel"/>
-    <xacro:wheel_link name="rear_left_wheel"/>
-    <xacro:wheel_link name="rear_right_wheel"/>
+    <xacro:mecanum_wheel name="front_left_wheel"/>
+    <xacro:mecanum_wheel name="front_right_wheel"/>
+    <xacro:mecanum_wheel name="rear_left_wheel"/>
+    <xacro:mecanum_wheel name="rear_right_wheel"/>
     <xacro:wheel_joint name="front_left_wheel_joint" parent="base_link" child="front_left_wheel" xyz="0.25 0.25 0"/>
     <xacro:wheel_joint name="front_right_wheel_joint" parent="base_link" child="front_right_wheel" xyz="0.25 -0.25 0"/>

Commit message: Tweak omniwheel geometry including rollers, and their positions to baselink

File: routewise_ws/src/rw_description/rw_description/urdf/mecanum_wheel.xacro (robot description, xacro)
@@ -2,10 +2,10 @@
 <robot xmlns:xacro="http://ros.org/wiki/xacro">
   <!-- Properties -->
-  <xacro:property name="wheel_mass" value="2.0"/> <!-- Assume a mass for the wheel -->
-  <xacro:property name="roller_mass" value="0.1"/> <!-- Assume a mass for the rollers -->
-  <xacro:property name="wheel_radius" value="0.1"/>
+  <xacro:property name="wheel_mass" value="2.0"/>
+  <xacro:property name="roller_mass" value="0.1"/>
+  <xacro:property name="wheel_radius" value="0.06"/>
   <xacro:property name="wheel_width" value="0.05"/>
-  <xacro:property name="roller_radius" value="0.02"/>
-  <xacro:property name="roller_length" value="0.05"/>
+  <xacro:property name="roller_radius" value="0.012"/>
+  <xacro:property name="roller_length" value="${wheel_width}"/>
   <xacro:property name="roller_angle" value="0.785398"/> <!-- 45 degrees in radians -->
   <!-- Mecanum Wheel Macro -->

File: routewise_ws/src/rw_description/rw_description/urdf/routewise_core.xacro (robot description, xacro)
@@ -5,4 +5,8 @@
     <xacro:property name="base_width" value="0.5"/>
     <xacro:property name="base_height" value="0.1"/>
+    <xacro:property name="width_offset_tolerance" value="0.008"/>
+    <!-- Derived Parameters -->
+    <xacro:property name="joint_offset_width" value="${base_width/2 + wheel_width/2 + width_offset_tolerance}"/>
+    <xacro:property name="joint_offset_length" value="${base_length/2}"/>
     <!-- Inertial Macros -->
     <xacro:macro name="inertial_box" params="mass x y z">
@@ -51,7 +55,7 @@
     <xacro:mecanum_wheel name="rear_left_wheel"/>
     <xacro:mecanum_wheel name="rear_right_wheel"/>
-    <xacro:wheel_joint name="front_left_wheel_joint" parent="base_link" child="front_left_wheel" xyz="0.25 0.25 0"/>
-    <xacro:wheel_joint name="front_right_wheel_joint" parent="base_link" child="front_right_wheel" xyz="0.25 -0.25 0"/>
-    <xacro:wheel_joint name="rear_left_wheel_joint" parent="base_link" child="rear_left_wheel" xyz="-0.25 0.25 0"/>
-    <xacro:wheel_joint name="rear_right_wheel_joint" parent="base_link" child="rear_right_wheel" xyz="-0.25 -0.25 0"/>
+    <xacro:wheel_joint name="front_left_wheel_joint" parent="base_link" child="front_left_wheel" xyz="${joint_offset_length} ${joint_offset_width} 0"/>
+    <xacro:wheel_joint name="front_right_wheel_joint" parent="base_link" child="front_right_wheel" xyz="${joint_offset_length} -${joint_offset_width} 0"/>
+    <xacro:wheel_joint name="rear_left_wheel_joint" parent="base_link" child="rear_left_wheel" xyz="-${joint_offset_length} ${joint_offset_width} 0"/>
+    <xacro:wheel_joint name="rear_right_wheel_joint" parent="base_link" child="rear_right_wheel" xyz="-${joint_offset_length} -${joint_offset_width} 0"/>
 </robot>

Commit message: Separate Mecanum wheel configurations based on roller angle inclinations

File: routewise_ws/src/rw_description/rw_description/urdf/mecanum_wheel.xacro (robot description, xacro)
@@ -8,7 +8,6 @@
   <xacro:property name="roller_radius" value="0.012"/>
   <xacro:property name="roller_length" value="${wheel_width}"/>
-  <xacro:property name="roller_angle" value="0.785398"/> <!-- 45 degrees in radians -->
   <!-- Mecanum Wheel Macro -->
-  <xacro:macro name="mecanum_wheel" params="name">
+  <xacro:macro name="mecanum_wheel" params="name roller_angle">
     <!-- Derived Properties -->
     <xacro:property name="I_wheel_xx_yy" value="0.0250833333333333"/>

File: routewise_ws/src/rw_description/rw_description/urdf/routewise_core.xacro (robot description, xacro)
@@ -46,13 +46,13 @@
             <parent link="${parent}"/>
             <child link="${child}"/>
-            <origin xyz="${xyz}" rpy="${pi/2} 0 0"/>
+            <origin xyz="${xyz}" rpy="${3*pi/2} 0 0"/>
             <axis xyz="0 0 1"/>
         </joint>
     </xacro:macro>
     <!-- Wheel Links and Joints -->
-    <xacro:mecanum_wheel name="front_left_wheel"/>
-    <xacro:mecanum_wheel name="front_right_wheel"/>
-    <xacro:mecanum_wheel name="rear_left_wheel"/>
-    <xacro:mecanum_wheel name="rear_right_wheel"/>
+    <xacro:mecanum_wheel name="front_left_wheel" roller_angle = "-0.785398"/> <!--Negative Inclination-->
+    <xacro:mecanum_wheel name="front_right_wheel" roller_angle = "0.785398"/> <!--Positive Inclination-->    <!-- 45 degrees in radians -->
+    <xacro:mecanum_wheel name="rear_left_wheel" roller_angle = "0.785398"/>
+    <xacro:mecanum_wheel name="rear_right_wheel" roller_angle = "-0.785398"/>
     <xacro:wheel_joint name="front_left_wheel_joint" parent="base_link" child="front_left_wheel" xyz="${joint_offset_length} ${joint_offset_width} 0"/>
     <xacro:wheel_joint name="front_right_wheel_joint" parent="base_link" child="front_right_wheel" xyz="${joint_offset_length} -${joint_offset_width} 0"/>
